File: pcb/MicroMouse_pcb_v1/MicroMouse_pcb_v1.kicad_pcb (KiCad board)
At the start: 2 copper layers, 100 x 90 mm, 16 parts, among them J1 USB_B_Micro, J2 Conn_01x20_Pin, J3 Conn_01x20_Pin, U2 ESP32-S3-WROOM-1, U3 AMS1117-3.3

Commit message: pcb progerss clock and breakout_board done
Parts:
- C1: value 100nF -> 0.1uF; footprint Capacitor_SMD:C_1206_3216Metric_Pad1.33x1.80mm_HandSolder -> Ivar_footprint_library:IVAR_1206_SMD_C
- C2, C3, C4: footprint Capacitor_SMD:C_1206_3216Metric_Pad1.33x1.80mm_HandSolder -> Ivar_footprint_library:IVAR_1206_SMD_C
- D1: value YELLOW -> 3.3v; footprint LED_SMD:LED_0603_1608Metric_Pad1.05x0.95mm_HandSolder -> Ivar_footprint_library:IVAR_0603_SMD_LED
- D2: value RED -> 5v; footprint LED_SMD:LED_0603_1608Metric_Pad1.05x0.95mm_HandSolder -> Ivar_footprint_library:IVAR_0603_SMD_LED
- F1: value 200mA -> 0.2A; footprint Fuse:Fuse_1206_3216Metric_Pad1.42x1.75mm_HandSolder -> Ivar_footprint_library:IVAR_1206_SMD_FUSE
- J2, J3: footprint Connector_PinSocket_2.54mm:PinSocket_1x20_P2.54mm_Vertical -> Connector_PinHeader_2.54mm:PinHeader_1x20_P2.54mm_Vertical
- Mico_USB_Breakout1: footprint Connector_PinSocket_2.54mm:PinSocket_1x05_P2.54mm_Vertical -> Ivar_footprint_library:IVAR_Micro_USB_breakout_board_5pin
- R1, R2: value R -> 1k; footprint Resistor_SMD:R_1206_3216Metric_Pad1.30x1.75mm_HandSolder -> Ivar_footprint_library:IVAR_1206_SMD_R
- R3: footprint Resistor_SMD:R_1206_3216Metric_Pad1.30x1.75mm_HandSolder -> Ivar_footprint_library:IVAR_1206_SMD_R
- moved U3 106.0 mm to (127.7, 104.5), turned to 90 degrees
- moved U2 106.0 mm to (128.2, 80.6)
- moved C3 104.2 mm to (137.6, 111.3), turned to 90 degrees
- moved C1 103.3 mm to (137.6, 107.9), turned to -90 degrees
- moved C4 100.5 mm to (122.2, 107.9), turned to -90 degrees
- moved R3 98.7 mm to (118.8, 104.3), turned to 90 degrees
- moved R1 95.3 mm to (137.6, 121.5), turned to -90 degrees
- moved F1 95.0 mm to (133.8, 104.3), turned to 90 degrees
- moved D1 91.5 mm to (137.6, 123.9), turned to 180 degrees
- moved J1 90.2 mm to (128.2, 122.1)
- moved C2 85.2 mm to (118.8, 111.3), turned to 90 degrees
- moved R2 77.6 mm to (118.8, 121.2), turned to -90 degrees
- moved D2 72.8 mm to (118.8, 123.9)
- moved Mico_USB_Breakout1 67.3 mm to (123.1, 112.8), turned to 90 degrees
- moved J2 62.5 mm to (114.2, 75.7)
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Connections:
- Mico_USB_Breakout1 pad 1: unconnected-(Mico_USB_Breakout1-Pin_1-Pad1) -> Net-(J1-VBUS)
- Mico_USB_Breakout1 pad 2: unconnected-(Mico_USB_Breakout1-Pin_2-Pad2) -> /DevBoard/USB_D_N
- Mico_USB_Breakout1 pad 3: unconnected-(Mico_USB_Breakout1-Pin_3-Pad3) -> /DevBoard/USB_D_P
- Mico_USB_Breakout1 pad 4: unconnected-(Mico_USB_Breakout1-Pin_4-Pad4) -> unconnected-(J1-ID-Pad4)
- Mico_USB_Breakout1 pad 5: unconnected-(Mico_USB_Breakout1-Pin_5-Pad5) -> GND
- U2 pad 13: /DevBoard/IO19 -> /DevBoard/USB_D_N
- U2 pad 14: /DevBoard/IO20 -> /DevBoard/USB_D_P
Routing:
- net /DevBoard/5v: track 0.00 -> 91.4 mm, vias 0 -> 1
- net /DevBoard/3.3v: track 0.00 -> 90.6 mm, vias 0 -> 4
- net /DevBoard/IO44: track 0.00 -> 50.7 mm, vias 0 -> 1
- net /DevBoard/IO43: track 0.00 -> 48.9 mm, vias 0 -> 1
- net /DevBoard/IO42: track 0.00 -> 43.4 mm, vias 0 -> 1
- net /DevBoard/IO15: track 0.00 -> 41.0 mm, vias 0 -> 2
- net /DevBoard/IO41: track 0.00 -> 39.7 mm, vias 0 -> 1
- net /DevBoard/EN: track 0.00 -> 39.4 mm, vias 0 -> 2
- net /DevBoard/USB_D_P: track 0.00 -> 36.7 mm, vias 0 -> 1
- net /DevBoard/USB_D_N: track 0.00 -> 35.9 mm, vias 0 -> 1
- net /DevBoard/IO40: track 0.00 -> 35.3 mm, vias 0 -> 1
- net /DevBoard/IO39: track 0.00 -> 33.0 mm, vias 0 -> 1
- net /DevBoard/IO14: track 0.00 -> 32.3 mm, vias 0 -> 1
- net /DevBoard/IO13: track 0.00 -> 29.3 mm, vias 0 -> 1
- net /DevBoard/IO2: track 0.00 -> 27.1 mm, vias 0 -> 1
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- added copper zone on B.Cu, net GND
- added copper zone on F.Cu, net GND
Other:
- board size 100 x 90 mm -> 100.2 x 90.3 mm
