File: pcb/breakout/breakout_pcb/breakout_pcb.kicad_sch (KiCad schematic)
At the start: 16 parts, among them J1 USB_B_Micro, J2 Conn_01x20_Pin, J3 Conn_01x20_Pin, U2 ESP32-S3-WROOM-1, U3 AMS1117-3.3

Commit message: pcb progerss clock and breakout_board done
Parts:
- renumbered C2 to C1, C1 to C2, D2 to D1, D1 to D2, R3 to R1, R1 to R3, U3 to U1
Changed lines of the file:
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@@
 		)
 		(instances
+			(project "breakout_pcb"
+				(path "/e5083fa8-0ef7-4956-b85b-f43be77f8073"
+					(reference "C3")
+					(unit 1)
+				)
+			)
 			(project "MicroMouse_pcb_v1"
 				(path "/edf27656-47bc-4351-b96d-7e76378cbc31/fd4eb493-81f4-493f-b2ab-0dc64d2656a2"
@@
 		(dnp no)
 		(fields_autoplaced yes)
-		(property "Reference" "#PWR04"
+		(property "Reference" "#PWR0105"
 			(at 58.42 116.84 0)
 			(effects
@@
 		)
 		(instances
+			(project "breakout_pcb"
+				(path "/e5083fa8-0ef7-4956-b85b-f43be77f8073"
+					(reference "#PWR0105")
+					(unit 1)
+				)
+			)
 			(project ""
 				(path "/edf27656-47bc-4351-b96d-7e76378cbc31/fd4eb493-81f4-493f-b2ab-0dc64d2656a2"
@@
 		)
 		(instances
+			(project "breakout_pcb"
+				(path "/e5083fa8-0ef7-4956-b85b-f43be77f8073"
+					(reference "F1")
+					(unit 1)
+				)
+			)
 			(project ""
 				(path "/edf27656-47bc-4351-b96d-7e76378cbc31/fd4eb493-81f4-493f-b2ab-0dc64d2656a2"
@@
 		(dnp no)
 		(fields_autoplaced yes)
-		(property "Reference" "U3"
+		(property "Reference" "U1"
 			(at 58.42 82.55 0)
 			(effects
@@
 		)
 		(instances
+			(project "breakout_pcb"
+				(path "/e5083fa8-0ef7-4956-b85b-f43be77f8073"
+					(reference "U1")
+					(unit 1)
+				)
+			)
 			(project ""
 				(path "/edf27656-47bc-4351-b96d-7e76378cbc31/fd4eb493-81f4-493f-b2ab-0dc64d2656a2"
@@
 		)
 		(instances
+			(project "breakout_pcb"
+				(path "/e5083fa8-0ef7-4956-b85b-f43be77f8073"
+					(reference "R2")
+					(unit 1)
+				)
+			)
 			(project "MicroMouse_pcb_v1"
 				(path "/edf27656-47bc-4351-b96d-7e76378cbc31/fd4eb493-81f4-493f-b2ab-0dc64d2656a2"
@@
 		(on_board yes)
 		(dnp no)
-		(property "Reference" "D2"
+		(property "Reference" "D1"
 			(at 252.984 44.704 90)
 			(effects
@@
 		)
 		(instances
+			(project "breakout_pcb"
+				(path "/e5083fa8-0ef7-4956-b85b-f43be77f8073"
+					(reference "D1")
+					(unit 1)
+				)
+			)
 			(project "MicroMouse_pcb_v1"
 				(path "/edf27656-47bc-4351-b96d-7e76378cbc31/fd4eb493-81f4-493f-b2ab-0dc64d2656a2"
@@
 		(dnp no)
 		(fields_autoplaced yes)
-		(property "Reference" "#PWR06"
+		(property "Reference" "#PWR0102"
 			(at 111.76 59.69 0)
 			(effects
@@
 		)
 		(instances
+			(project "breakout_pcb"
+				(path "/e5083fa8-0ef7-4956-b85b-f43be77f8073"
+					(reference "#PWR0102")
+					(unit 1)
+				)
+			)
 			(project ""
 				(path "/edf27656-47bc-4351-b96d-7e76378cbc31/fd4eb493-81f4-493f-b2ab-0dc64d2656a2"
@@
 		(dnp no)
 		(fields_autoplaced yes)
-		(property "Reference" "#PWR010"
+		(property "Reference" "#PWR0107"
 			(at 171.45 167.64 0)
 			(effects
@@
 		)
 		(instances
+			(project "breakout_pcb"
+				(path "/e5083fa8-0ef7-4956-b85b-f43be77f8073"
+					(reference "#PWR0107")
+					(unit 1)
+				)
+			)
 			(project ""
 				(path "/edf27656-47bc-4351-b96d-7e76378cbc31/fd4eb493-81f4-493f-b2ab-0dc64d2656a2"
@@
 		(on_board yes)
 		(dnp no)
-		(property "Reference" "#PWR09"
+		(property "Reference" "#PWR0103"
 			(at 120.65 167.64 0)
 			(effects
@@
 		)
 		(instances
+			(project "breakout_pcb"
+				(path "/e5083fa8-0ef7-4956-b85b-f43be77f8073"
+					(reference "#PWR0103")
+					(unit 1)
+				)
+			)
 			(project "MicroMouse_pcb_v1"
 				(path "/edf27656-47bc-4351-b96d-7e76378cbc31/fd4eb493-81f4-493f-b2ab-0dc64d2656a2"
@@
 		(on_board yes)
 		(dnp no)
-		(property "Reference" "#PWR07"
+		(property "Reference" "#PWR0104"
 			(at 119.38 123.19 0)
 			(effects
@@
 		)
 		(instances
+			(project "breakout_pcb"
+				(path "/e5083fa8-0ef7-4956-b85b-f43be77f8073"
+					(reference "#PWR0104")
+					(unit 1)
+				)
+			)
 			(project ""
 				(path "/edf27656-47bc-4351-b96d-7e76378cbc31/fd4eb493-81f4-493f-b2ab-0dc64d2656a2"
@@
 		(dnp no)
 		(fields_autoplaced yes)
-		(property "Reference" "#PWR01"
+		(property "Reference" "#PWR0109"
 			(at 262.89 59.69 0)
 			(effects
@@
 		)
 		(instances
+			(project "breakout_pcb"
+				(path "/e5083fa8-0ef7-4956-b85b-f43be77f8073"
+					(reference "#PWR0109")
+					(unit 1)
+				)
+			)
 			(project ""
 				(path "/edf27656-47bc-4351-b96d-7e76378cbc31/fd4eb493-81f4-493f-b2ab-0dc64d2656a2"
@@
 		(on_board yes)
 		(dnp no)
-		(property "Reference" "R1"
+		(property "Reference" "R3"
 			(at 264.414 34.29 0)
 			(effects
@@
 		)
 		(instances
+			(project "breakout_pcb"
+				(path "/e5083fa8-0ef7-4956-b85b-f43be77f8073"
+					(reference "R3")
+					(unit 1)
+				)
+			)
 			(project ""
 				(path "/edf27656-47bc-4351-b96d-7e76378cbc31/fd4eb493-81f4-493f-b2ab-0dc64d2656a2"
@@
 		(on_board yes)
 		(dnp no)
-		(property "Reference" "C1"
+		(property "Reference" "C2"
 			(at 48.514 95.25 0)
 			(effects
@@
 		)
 		(instances
+			(project "breakout_pcb"
+				(path "/e5083fa8-0ef7-4956-b85b-f43be77f8073"
+					(reference "C2")
+					(unit 1)
+				)
+			)
 			(project ""
 				(path "/edf27656-47bc-4351-b96d-7e76378cbc31/fd4eb493-81f4-493f-b2ab-0dc64d2656a2"
@@
 		(on_board yes)
 		(dnp no)
-		(property "Reference" "C2"
+		(property "Reference" "C1"
 			(at 29.464 95.758 0)
 			(effects
@@
 		)
 		(instances
+			(project "breakout_pcb"
+				(path "/e5083fa8-0ef7-4956-b85b-f43be77f8073"
+					(reference "C1")
+					(unit 1)
+				)
+			)
 			(project "MicroMouse_pcb_v1"
 				(path "/edf27656-47bc-4351-b96d-7e76378cbc31/fd4eb493-81f4-493f-b2ab-0dc64d2656a2"
@@
 		)
 		(instances
+			(project "breakout_pcb"
+				(path "/e5083fa8-0ef7-4956-b85b-f43be77f8073"
+					(reference "J2")
+					(unit 1)
+				)
+			)
 			(project ""
 				(path "/edf27656-47bc-4351-b96d-7e76378cbc31/fd4eb493-81f4-493f-b2ab-0dc64d2656a2"
@@
 		(dnp no)
 		(fields_autoplaced yes)
-		(property "Reference" "#PWR03"
+		(property "Reference" "#PWR0101"
 			(at 35.56 71.12 0)
 			(effects
@@
 		)
 		(instances
+			(project "breakout_pcb"
+				(path "/e5083fa8-0ef7-4956-b85b-f43be77f8073"
+					(reference "#PWR0101")
+					(unit 1)
+				)
+			)
 			(project ""
 				(path "/edf27656-47bc-4351-b96d-7e76378cbc31/fd4eb493-81f4-493f-b2ab-0dc64d2656a2"
@@
 		)
 		(instances
+			(project "breakout_pcb"
+				(path "/e5083fa8-0ef7-4956-b85b-f43be77f8073"
+					(reference "Mico_USB_Breakout1")
+					(unit 1)
+				)
+			)
 			(project ""
 				(path "/edf27656-47bc-4351-b96d-7e76378cbc31/fd4eb493-81f4-493f-b2ab-0dc64d2656a2"
@@
 		(on_board yes)
 		(dnp no)
-		(property "Reference" "#PWR08"
+		(property "Reference" "#PWR0108"
 			(at 172.72 123.19 0)
 			(effects
@@
 		)
 		(instances
+			(project "breakout_pcb"
+				(path "/e5083fa8-0ef7-4956-b85b-f43be77f8073"
+					(reference "#PWR0108")
+					(unit 1)
+				)
+			)
 			(project "MicroMouse_pcb_v1"
 				(path "/edf27656-47bc-4351-b96d-7e76378cbc31/fd4eb493-81f4-493f-b2ab-0dc64d2656a2"
@@
 		)
 		(instances
+			(project "breakout_pcb"
+				(path "/e5083fa8-0ef7-4956-b85b-f43be77f8073"
+					(reference "C4")
+					(unit 1)
+				)
+			)
 			(project "MicroMouse_pcb_v1"
 				(path "/edf27656-47bc-4351-b96d-7e76378cbc31/fd4eb493-81f4-493f-b2ab-0dc64d2656a2"
@@
 		)
 		(instances
+			(project "breakout_pcb"
+				(path "/e5083fa8-0ef7-4956-b85b-f43be77f8073"
+					(reference "J1")
+					(unit 1)
+				)
+			)
 			(project ""
 				(path "/edf27656-47bc-4351-b96d-7e76378cbc31/fd4eb493-81f4-493f-b2ab-0dc64d2656a2"
@@
 		)
 		(instances
+			(project "breakout_pcb"
+				(path "/e5083fa8-0ef7-4956-b85b-f43be77f8073"
+					(reference "U2")
+					(unit 1)
+				)
+			)
 			(project ""
 				(path "/edf27656-47bc-4351-b96d-7e76378cbc31/fd4eb493-81f4-493f-b2ab-0dc64d2656a2"
@@
 		)
 		(instances
+			(project "breakout_pcb"
+				(path "/e5083fa8-0ef7-4956-b85b-f43be77f8073"
+					(reference "J3")
+					(unit 1)
+				)
+			)
 			(project "MicroMouse_pcb_v1"
 				(path "/edf27656-47bc-4351-b96d-7e76378cbc31/fd4eb493-81f4-493f-b2ab-0dc64d2656a2"
@@
 		(dnp no)
 		(fields_autoplaced yes)
-		(property "Reference" "#PWR02"
+		(property "Reference" "#PWR0110"
 			(at 251.46 59.69 0)
 			(effects
@@
 		)
 		(instances
+			(project "breakout_pcb"
+				(path "/e5083fa8-0ef7-4956-b85b-f43be77f8073"
+					(reference "#PWR0110")
+					(unit 1)
+				)
+			)
 			(project "MicroMouse_pcb_v1"
 				(path "/edf27656-47bc-4351-b96d-7e76378cbc31/fd4eb493-81f4-493f-b2ab-0dc64d2656a2"
@@
 		(dnp no)
 		(fields_autoplaced yes)
-		(property "Reference" "#PWR05"
+		(property "Reference" "#PWR0106"
 			(at 146.05 102.87 0)
 			(effects
@@
 		)
 		(instances
+			(project "breakout_pcb"
+				(path "/e5083fa8-0ef7-4956-b85b-f43be77f8073"
+					(reference "#PWR0106")
+					(unit 1)
+				)
+			)
 			(project ""
 				(path "/edf27656-47bc-4351-b96d-7e76378cbc31/fd4eb493-81f4-493f-b2ab-0dc64d2656a2"
@@
 		(on_board yes)
 		(dnp no)
-		(property "Reference" "D1"
+		(property "Reference" "D2"
 			(at 264.668 44.704 90)
 			(effects
@@
 		)
 		(instances
+			(project "breakout_pcb"
+				(path "/e5083fa8-0ef7-4956-b85b-f43be77f8073"
+					(reference "D2")
+					(unit 1)
+				)
+			)
 			(project ""
 				(path "/edf27656-47bc-4351-b96d-7e76378cbc31/fd4eb493-81f4-493f-b2ab-0dc64d2656a2"
@@
 		(on_board yes)
 		(dnp no)
-		(property "Reference" "R3"
+		(property "Reference" "R1"
 			(at 113.284 36.83 0)
 			(effects
@@
 		)
 		(instances
+			(project "breakout_pcb"
+				(path "/e5083fa8-0ef7-4956-b85b-f43be77f8073"
+					(reference "R1")
+					(unit 1)
+				)
+			)
 			(project "MicroMouse_pcb_v1"
 				(path "/edf27656-47bc-4351-b96d-7e76378cbc31/fd4eb493-81f4-493f-b2ab-0dc64d2656a2"
@@
 		)
 	)
+	(sheet_instances
+		(path "/"
+			(page "1")
+		)
+	)
